File: HAT PCB/SSS_HAT.kicad_sch (KiCad schematic)
At the start: 21 parts, among them J1 ESP32_Connector_0, J2 ESP32_Connector_1, J3 I2C, J4 I2C, J5 I2C, J6 ADC, U1 TJA1051T, U2 ADS8320EB_250, U3 ICM-42688-P

Commit message: Fixed J1 & J2 footprints which called for an entire re-route
Parts:
- added C10, C11, C12, C13, C14, C15, C16, C17, C18, C19, C20, C21, C22, C23, C24, C25, C7, C8, C9: 10nF, Capacitor_SMD:C_0201_0603Metric, symbol Device:C
- added J7: WS, Connector_Hirose:Hirose_DF3EA-03P-2H_1x03-1MP_P2.00mm_Horizontal, symbol Connector_Generic_MountingPin:Conn_01x03_MountingPin
- added R10, R11, R12, R13, R14, R15, R16, R17, R18, R19, R20, R21, R22, R3, R4, R5, R6, R7, R8, R9: 1k, Capacitor_SMD:C_0201_0603Metric, symbol Device:R_Small
- C6: value 1μF -> 10nF; footprint Capacitor_SMD:C_0402_1005Metric_Pad0.74x0.62mm_HandSolder -> Capacitor_SMD:C_0201_0603Metric
- J1: footprint Connector_PinSocket_1.27mm:PinSocket_1x22_P1.27mm_Vertical_SMD_Pin1Left -> Connector_PinSocket_2.54mm:PinSocket_1x22_P2.54mm_Vertical
- J2: footprint Connector_PinSocket_1.27mm:PinSocket_1x22_P1.27mm_Vertical_SMD_Pin1Right -> Connector_PinSocket_2.54mm:PinSocket_1x22_P2.54mm_Vertical
- renumbered C4 to C3, C3 to C4
Connections:
- net +5V: now also J7.1 (Pin_1)
- net A_In: now also J6.2 (Pin_2), R3.2; no longer C6.1, J2.4 (Pin_4), J6.3 (Pin_3), U2.2 (+IN)
- net GND: now also C6.1, J6.3 (Pin_3), C10.1, C11.1, C12.1, C13.1, C14.1, C15.1, C16.1, C17.1, C18.1, C19.1, C20.1, C21.1, C22.1, C23.1, C24.1, C25.1, C7.1, C8.1, C9.1, J7.3 (Pin_3), J7.MP (MountPin); no longer C6.2, J6.2 (Pin_2)
- net WS_IN: now reaches J1.7 (Pin_7)
- net WS_IN: now also J7.2 (Pin_2)
- new net: C17.2, R14.1, R15.2
- new net: C21.2, R18.1, R19.2
- new net: C20.2, R17.1, R18.2
- new net: C9.2, R6.1, R7.2
- new net: C8.2, R5.1, R6.2
- new net: C13.2, R10.1, R11.2
- new net: C12.2, R10.2, R9.1
- new net: C7.2, R4.1, R5.2
- new net: C6.2, R3.1, R4.2
- new net: C24.2, R21.1, R22.2
- new net: C15.2, R12.1, R13.2
- new net: C11.2, R8.1, R9.2
- new net: C16.2, R13.1, R14.2
- new net: C19.2, R16.1, R17.2
- new net: C18.2, R15.1, R16.2
- new net: C23.2, R20.1, R21.2
- new net: C10.2, R7.1, R8.2
- new net: C14.2, R11.1, R12.2
- new net: C22.2, R19.1, R20.2
- new net AA_out: C25.2, J2.4 (Pin_4), R22.1, U2.2 (+IN)
- no-connect marks 25 -> 24
Other:
- note added: "Wheel speed input"
