File: HAT PCB/SSS_HAT.kicad_pcb (KiCad board)
At the start: 4 copper layers, 120.2 x 30.4 mm, 64 parts, among them J1 ESP32_Connector_0, J2 ESP32_Connector_1, J3 I2C, J4 I2C, J5 I2C, J6 ADC, J7 WS, U1 TJA1051T, U2 ADS8320EB_250, U3 ICM-42688-P

Commit message: added updates from 11/5 meeting. Faraday cage WIP
Routing:
- net +5V: track 146.5 -> 15.0 mm, vias 5 -> 7
- net A_In: track 14.1 -> 15.8 mm
- net GND: vias 28 -> 93
- added copper zone on In1.Cu, net +3.3V
- added copper zone on B.Cu, net +5V
- added copper zone on In2.Cu, net GND
- removed copper zone on In2.Cu, net +3.3V
- removed copper zone on In1.Cu, net GND
