File: SUS/SUS.kicad_pcb (KiCad board)
At the start: 4 copper layers, 58 x 64 mm, 67 parts, among them J1 ESP32_Connector_0, J2 ESP32_Connector_1, J3 D25P13A4GV00LF, U1 HT7333, U2 ADS1015IDGSR, U3 ICM-42688-P, U5 SN65HVD232

Commit message: Minor Changes
Parts:
- U1: value HT7333 -> HT7350-A
- renumbered U5 to U4
Changed lines of the file:
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@@
 	(net 69 "unconnected-(J3-Pad25)")
 	(net 70 "unconnected-(U2-AIN1-Pad5)")
-	(net 71 "unconnected-(U5-NC-Pad5)")
-	(net 72 "unconnected-(U5-NC-Pad8)")
+	(net 71 "unconnected-(U4-NC-Pad5)")
+	(net 72 "unconnected-(U4-NC-Pad8)")
 	(net 73 "unconnected-(J1-Pin_7-Pad7)")
 	(net 74 "unconnected-(J1-Pin_6-Pad6)")
@@
 			(net 66 "unconnected-(J3-Pad21)")
 			(pinfunction "21")
-			(pintype "unspecified")
+			(pintype "unspecified+no_connect")
 		)
 		(pad "22" thru_hole circle
@@
 			(net 67 "unconnected-(J3-Pad24)")
 			(pinfunction "24")
-			(pintype "unspecified")
+			(pintype "unspecified+no_connect")
 		)
 		(pad "25" thru_hole circle
@@
 			(net 69 "unconnected-(J3-Pad25)")
 			(pinfunction "25")
-			(pintype "unspecified")
+			(pintype "unspecified+no_connect")
 		)
 	)
@@
 			)
 		)
-		(property "Value" "HT7333"
+		(property "Value" "HT7350-A"
 			(at 3.19 4.435 90)
 			(layer "F.Fab")
@@
 		(descr "SOIC, 8 Pin (JEDEC MS-012AA, https://www.analog.com/media/en/package-pcb-resources/package/pkg_pdf/soic_narrow-r/r_8.pdf), generated with kicad-footprint-generator ipc_gullwing_generator.py")
 		(tags "SOIC SO")
-		(property "Reference" "U5"
+		(property "Reference" "U4"
 			(at 0.02 4.02 180)
 			(layer "F.SilkS")
@@
 			(layers "F.Cu" "F.Paste" "F.Mask")
 			(roundrect_rratio 0.25)
-			(net 71 "unconnected-(U5-NC-Pad5)")
+			(net 71 "unconnected-(U4-NC-Pad5)")
 			(pinfunction "NC")
 			(pintype "no_connect")
@@
 			(layers "F.Cu" "F.Paste" "F.Mask")
 			(roundrect_rratio 0.25)
-			(net 72 "unconnected-(U5-NC-Pad8)")
+			(net 72 "unconnected-(U4-NC-Pad8)")
 			(pinfunction "NC")
 			(pintype "no_connect")
@@
 			(net 76 "unconnected-(J1-Pin_4-Pad4)")
 			(pinfunction "Pin_4")
-			(pintype "passive")
+			(pintype "passive+no_connect")
 		)
 		(pad "5" thru_hole oval
@@
 			(net 75 "unconnected-(J1-Pin_5-Pad5)")
 			(pinfunction "Pin_5")
-			(pintype "passive")
+			(pintype "passive+no_connect")
 		)
 		(pad "6" thru_hole oval
@@
 			(net 8 "unconnected-(J1-Pin_9-Pad9)")
 			(pinfunction "Pin_9")
-			(pintype "passive")
+			(pintype "passive+no_connect")
 		)
 		(pad "10" thru_hole oval
@@
 			(net 23 "unconnected-(J1-Pin_10-Pad10)")
 			(pinfunction "Pin_10")
-			(pintype "passive")
+			(pintype "passive+no_connect")
 		)
 		(pad "11" thru_hole oval

Commit message: Added jumpers for 5v and 3v3 for lin pot
Parts:
- added JP2: SolderJumper_2_Open, Jumper:SolderJumper-2_P1.3mm_Open_TrianglePad1.0x1.5mm, B.Cu at (132.5, 54.4)
- added JP3: SolderJumper_2_Open, Jumper:SolderJumper-2_P1.3mm_Open_TrianglePad1.0x1.5mm, B.Cu at (132.5, 58.0)
- JP1: moved to B.Cu
Connections:
- J3 pad 16: +5V -> Net-(JP2-B)
Routing:
- net Net-(JP2-B): track 0.00 -> 26.6 mm
- net +5V: track 2.12 -> 4.14 mm, vias 1 -> 2
- net +3.3V: track 13.4 -> 14.9 mm, vias 6 -> 7
- net AA_out: track 19.2 -> 19.3 mm, vias 0 -> 1
